File: 514 pcb design/514 pcb design.kicad_pcb (KiCad board)
At the start: 2 copper layers, 1 part

Commit message: Update
Parts:
- added A1: Arduino_Nano_ESP32_Tile, esp32_footprint:Arduino_Nano_ESP32_Tile, F.Cu at (75.6, 90.2)
- added Brd1: SSD1306, ssd1306:128x64OLED, F.Cu at (77.7, 105.0)
- added U1: HC-SR04, HC-SR04:XCVR_HC-SR04, F.Cu at (62.4, 25.7)
- added U2: OV7670, OV7670:OV7670, F.Cu at (39.9, 68.1)
- moved A2 34.3 mm to (99.3, 90.2)
Connections:
- A2 pad 3V3: unconnected-(A2-3.3V-Pad3V3) -> Net-(A2-3.3V)
- A2 pad A4: unconnected-(A2-A4/SDA-PadA4) -> Net-(A2-A4/SDA)
- A2 pad A5: unconnected-(A2-A5/SCL-PadA5) -> Net-(A2-A5/SCL)
- A2 pad D2: unconnected-(A2-PadD2) -> Net-(D1-A)
- A2 pad GND1: unconnected-(A2-GND-PadGND1) -> Net-(Brd1-GND)
- A2 pad GND2: unconnected-(A2-GND-PadGND2) -> Net-(D1-BK)

Commit message: update
Parts:
- removed A1: Arduino_Nano_ESP32_Tile, esp32_footprint:Arduino_Nano_ESP32_Tile
- removed U1: HC-SR04, HC-SR04:XCVR_HC-SR04
- removed U2: OV7670, OV7670:OV7670
- added BT1: Battery_Cell, Connector_JST:JST_PHD_B8B-PHDSS_2x04_P2.00mm_Vertical, F.Cu at (92.7, 58.4)
- added D1: LED_RGBA, LED_SMD:LED_SK6812_PLCC4_5.0x5.0mm_P3.2mm, F.Cu at (99.2, 99.1)
- added D2: LED, LED_SMD:LED_0805_2012Metric_Pad1.15x1.40mm_HandSolder, F.Cu at (109.2, 61.0)
- added J1: Conn_01x02_Pin, Connector_JST:JST_XA_B02B-XASK-1-A_1x02_P2.50mm_Vertical, F.Cu at (109.2, 100.3)
- added M1: Stepper_Motor_bipolar, x27_footprint:x27_stepper, F.Cu at (161.3, 101.6)
- added R1: 85Ω, Resistor_SMD:R_0805_2012Metric_Pad1.20x1.40mm_HandSolder, F.Cu at (109.2, 108.0)
- added R2: 85Ω, Resistor_SMD:R_0805_2012Metric_Pad1.20x1.40mm_HandSolder, F.Cu at (116.8, 61.0)
- added SW1: SW_SPDT, Connector_JST:JST_EH_B3B-EH-A_1x03_P2.50mm_Vertical, F.Cu at (130.8, 61.0)
- moved A2 36.2 mm to (128.3, 68.6), turned to 180 degrees
- moved Brd1 33.4 mm to (98.9, 79.2)
Connections:
- net Net-(A2-3.3V) renamed /3v3
- net Net-(A2-A4/SDA) renamed /SDA
- net Net-(A2-A5/SCL) renamed /SCL
- A2 pad A0: unconnected-(A2-PadA0) -> /A0
- A2 pad A1: unconnected-(A2-PadA1) -> /A1
- A2 pad D2: Net-(D1-A) -> /D2
- A2 pad D3: unconnected-(A2-PadD3) -> /D3
- A2 pad D4: unconnected-(A2-PadD4) -> /D4
- A2 pad D8: unconnected-(A2-PadD8) -> /D8
- A2 pad D9: unconnected-(A2-PadD9) -> /D9
- A2 pad GND1: Net-(Brd1-GND) -> unconnected-(A2-GND-PadGND1)
- A2 pad GND2: Net-(D1-BK) -> GND
- A2 pad VIN: unconnected-(A2-PadVIN) -> /Vin
- Brd1 pad 1: Net-(Brd1-GND) -> GND
Routing:
- net GND: track 0.00 -> 81.6 mm
- net /Vin: track 0.00 -> 67.4 mm
- net /D8: track 0.00 -> 37.6 mm
- net Net-(BT1-+): track 0.00 -> 37.5 mm
- net /D9: track 0.00 -> 36.1 mm
- net /D2: track 0.00 -> 32.8 mm
- net /SCL: track 0.00 -> 31.8 mm
- net /SDA: track 0.00 -> 28.2 mm
- net /3v3: track 0.00 -> 24.7 mm
- net Net-(D1-A): track 0.00 -> 14.5 mm
- net /D4: track 0.00 -> 11.6 mm
- net /D3: track 0.00 -> 9.53 mm
- net Net-(SW1-C): track 0.00 -> 9.38 mm
- net Net-(D2-A): track 0.00 -> 7.63 mm
- net unconnected-(A2-GND-PadGND1): track 0.00 -> 0.64 mm
- added copper zone on B.Cu, net GND
- added copper zone on F.Cu, net GND
Other:
- board outline added: 91.4 x 61 mm
- board text added: "ZIA 514 PCBdesign V1.0"
