File: 514 pcb design/514 pcb design.kicad_sch (KiCad schematic)
At the start: 1 part

Commit message: Update
Parts:
- added A1: Arduino_Nano_ESP32_Tile, esp32_footprint:Arduino_Nano_ESP32_Tile, symbol arduino-library:Arduino_Nano_ESP32_Tile
- added Brd1: SSD1306, ssd1306:128x64OLED, symbol SSD1306-128x64_OLED:SSD1306
- added D1: LED_RGBA, symbol Device:LED_RGBA
- added U1: HC-SR04, HC-SR04:XCVR_HC-SR04, symbol HC-SR04:HC-SR04
- added U2: OV7670, OV7670:OV7670, symbol OV7670:OV7670
Connections:
- net at A2.3V3 (3.3V): now also Brd1.2 (VCC)
- net at A2.A4 (A4/SDA): now also Brd1.4 (SDA)
- net at A2.A5 (A5/SCL): now also Brd1.3 (SCL)
- net at A2.D2: now also D1.4 (A)
- net at A2.GND1 (GND): now also Brd1.1 (GND)
- net at A2.GND2 (GND): now also D1.1 (RK), D1.2 (GK), D1.3 (BK)
- new net: A1.D10, U2.D1
- new net: A1.D9, U2.D3
- new net: A1.D8, U2.D5
- new net: A1.D7, U2.D7
- new net: A1.GND2 (GND), U1.4 (GND), U2.GND
- new net: A1.A5 (A5/SCL), U2.SCL
- new net: A1.A4 (A4/SDA), U2.SDA
- new net: A1.3V3 (3.3V), U1.1 (VCC), U2.VCC
- new net: A1.A0, U1.2 (TRIG)
- new net: A1.A1, U1.3 (ECHO)
Other:
- moved on the sheet: A2

Commit message: update
Parts:
- removed A1: Arduino_Nano_ESP32_Tile, esp32_footprint:Arduino_Nano_ESP32_Tile, symbol arduino-library:Arduino_Nano_ESP32_Tile
- removed U1: HC-SR04, HC-SR04:XCVR_HC-SR04, symbol HC-SR04:HC-SR04
- removed U2: OV7670, OV7670:OV7670, symbol OV7670:OV7670
- added BT1: Battery_Cell, Connector_JST:JST_PHD_B8B-PHDSS_2x04_P2.00mm_Vertical, symbol Device:Battery_Cell
- added D2: LED, LED_SMD:LED_0805_2012Metric_Pad1.15x1.40mm_HandSolder, symbol Device:LED
- added J1: Conn_01x02_Pin, Connector_JST:JST_XA_B02B-XASK-1-A_1x02_P2.50mm_Vertical, symbol Connector:Conn_01x02_Pin
- added M1: Stepper_Motor_bipolar, x27_footprint:x27_stepper, symbol Motor:Stepper_Motor_bipolar
- added R1, R2: 85Ω, Resistor_SMD:R_0805_2012Metric_Pad1.20x1.40mm_HandSolder, symbol Device:R
- added SW1: SW_SPDT, Connector_JST:JST_EH_B3B-EH-A_1x03_P2.50mm_Vertical, symbol Switch:SW_SPDT
- D1: footprint (none) -> LED_SMD:LED_SK6812_PLCC4_5.0x5.0mm_P3.2mm
Connections:
- net 3v3: now reaches A2.3V3 (3.3V), Brd1.2 (VCC)
- net A0: now reaches A2.A0
- net A1: now reaches A2.A1
- net SDA: now reaches A2.A4 (A4/SDA), Brd1.4 (SDA)
- net SCL: now reaches A2.A5 (A5/SCL), Brd1.3 (SCL)
- net at D1.4 (A): now also R1.1; no longer A2.D2
- net D3: now reaches A2.D3
- net D3: now also M1.3
- net D4: now reaches A2.D4
- net D4: now also M1.4
- net D8: now reaches A2.D8
- net D8: now also M1.2 (-)
- net D9: now reaches A2.D9
- net D9: now also M1.1
- net at A2.GND1 (GND): no longer Brd1.1 (GND)
- net GND: now reaches A2.GND2 (GND), D1.1 (RK), D1.2 (GK), D1.3 (BK)
- net GND: now also Brd1.1 (GND), BT1.2 (-), D2.1 (K), J1.2 (Pin_2)
- net Vin: now reaches A2.VIN
- net Vin: now also J1.1 (Pin_1), SW1.1 (A)
- new net: BT1.1 (+), SW1.2 (B)
- new net: R2.2, SW1.3 (C)
- new net: D2.2 (A), R2.1
- new net D2: A2.D2, R1.2
- no-connect marks 0 -> 18
Other:
- company: (none) -> Zia Sun
- title: (none) -> stepper motor demo
- moved on the sheet: A2, Brd1, D1
